File: KiCad/AXOLORACK.sch (KiCad schematic (older format))
At the start: 19 parts, among them J1 Conn_01x37_Axolot, J2 Eurorack, J3 Conn_02x03_Counter_Clockwise, SW1 Rotary_Encoder_Switch

Commit message: Update AXOLORACK.sch
Parts:
- added R3, R4: 10K, symbol Device:R
Connections:
- net PB6: now also R4.2
- net PB7: now also R3.2
- net VDD: now also R3.1, R4.1
Other:
- note added: "AxoloRack - Another EurorAxoloti\n"
- moved on the sheet: J2
Changed lines of the file:
@@
 EESchema Schematic File Version 4
+LIBS:AXOLORACK-cache
 EELAYER 30 0
 EELAYER END
@@
 L Connector_Generic:Conn_02x05_Counter_Clockwise J2
 U 1 1 5DF5972D
-P 6000 7000
-F 0 "J2" H 6050 7417 50  0000 C CNN
-F 1 "Eurorack" H 6050 7326 50  0000 C CNN
-F 2 "" H 6000 7000 50  0001 C CNN
-F 3 "~" H 6000 7000 50  0001 C CNN
-	1    6000 7000
+P 1200 7000
+F 0 "J2" H 1250 7417 50  0000 C CNN
+F 1 "Eurorack" H 1250 7326 50  0000 C CNN
+F 2 "" H 1200 7000 50  0001 C CNN
+F 3 "~" H 1200 7000 50  0001 C CNN
+	1    1200 7000
 	1    0    0    -1
 $EndComp
@@
 L power:GND #PWR0108
 U 1 1 5DF5A893
-P 6550 7000
-F 0 "#PWR0108" H 6550 6750 50  0001 C CNN
-F 1 "GND" H 6555 6827 50  0000 C CNN
-F 2 "" H 6550 7000 50  0001 C CNN
-F 3 "" H 6550 7000 50  0001 C CNN
-	1    6550 7000
-	1    0    0    -1
-$EndComp
-Wire Wire Line
-	6350 7000 6350 6900
-Wire Wire Line
-	6350 6900 6300 6900
-Wire Wire Line
-	6300 7000 6350 7000
-Wire Wire Line
-	6350 7000 6350 7100
-Wire Wire Line
-	6350 7100 6300 7100
-Connection ~ 6350 7000
+P 1750 7000
+F 0 "#PWR0108" H 1750 6750 50  0001 C CNN
+F 1 "GND" H 1755 6827 50  0000 C CNN
+F 2 "" H 1750 7000 50  0001 C CNN
+F 3 "" H 1750 7000 50  0001 C CNN
+	1    1750 7000
+	1    0    0    -1
+$EndComp
+Wire Wire Line
+	1550 7000 1550 6900
+Wire Wire Line
+	1550 6900 1500 6900
+Wire Wire Line
+	1500 7000 1550 7000
+Wire Wire Line
+	1550 7000 1550 7100
+Wire Wire Line
+	1550 7100 1500 7100
+Connection ~ 1550 7000
 $Comp
 L power:GND #PWR0112
 U 1 1 5DF671BA
-P 5650 7000
-F 0 "#PWR0112" H 5650 6750 50  0001 C CNN
-F 1 "GND" H 5655 6827 50  0000 C CNN
-F 2 "" H 5650 7000 50  0001 C CNN
-F 3 "" H 5650 7000 50  0001 C CNN
-	1    5650 7000
-	1    0    0    -1
-$EndComp
-Wire Wire Line
-	5800 7100 5750 7100
-Wire Wire Line
-	5750 7100 5750 7000
-Wire Wire Line
-	5750 6900 5800 6900
-Connection ~ 5750 7000
-Wire Wire Line
-	5750 7000 5800 7000
-Wire Wire Line
-	5750 7000 5750 6900
-Wire Wire Line
-	6300 6800 6400 6800
-Wire Wire Line
-	6400 6800 6400 6700
-Wire Wire Line
-	6400 6700 6600 6700
+P 850 7000
+F 0 "#PWR0112" H 850 6750 50  0001 C CNN
+F 1 "GND" H 855 6827 50  0000 C CNN
+F 2 "" H 850 7000 50  0001 C CNN
+F 3 "" H 850 7000 50  0001 C CNN
+	1    850  7000
+	1    0    0    -1
+$EndComp
+Wire Wire Line
+	1000 7100 950  7100
+Wire Wire Line
+	950  7100 950  7000
+Wire Wire Line
+	950  6900 1000 6900
+Connection ~ 950  7000
+Wire Wire Line
+	950  7000 1000 7000
+Wire Wire Line
+	950  7000 950  6900
+Wire Wire Line
+	1500 6800 1600 6800
+Wire Wire Line
+	1600 6800 1600 6700
+Wire Wire Line
+	1600 6700 1800 6700
 $Comp
 L power:+12V #PWR0113
 U 1 1 5DF8509E
-P 6600 6700
-F 0 "#PWR0113" H 6600 6550 50  0001 C CNN
-F 1 "+12V" H 6615 6873 50  0000 C CNN
-F 2 "" H 6600 6700 50  0001 C CNN
-F 3 "" H 6600 6700 50  0001 C CNN
-	1    6600 6700
-	1    0    0    -1
-$EndComp
-Wire Wire Line
-	6350 7000 6550 7000
-Wire Wire Line
-	5650 7000 5750 7000
+P 1800 6700
+F 0 "#PWR0113" H 1800 6550 50  0001 C CNN
+F 1 "+12V" H 1815 6873 50  0000 C CNN
+F 2 "" H 1800 6700 50  0001 C CNN
+F 3 "" H 1800 6700 50  0001 C CNN
+	1    1800 6700
+	1    0    0    -1
+$EndComp
+Wire Wire Line
+	1550 7000 1750 7000
+Wire Wire Line
+	850  7000 950  7000
 $Comp
 L MyLib:Conn_01x37_Axolot J1
@@
 	2050 2900 2050 2500
 Wire Wire Line
-	5800 6800 5750 6800
-Wire Wire Line
-	5750 6800 5750 6700
-Wire Wire Line
-	5750 6700 5650 6700
-Wire Wire Line
-	5800 7200 5750 7200
-Wire Wire Line
-	5750 7200 5750 7300
-Text Label 6400 6750 0    28   ~ 0
+	1000 6800 950  6800
+Wire Wire Line
+	950  6800 950  6700
+Wire Wire Line
+	950  6700 850  6700
+Wire Wire Line
+	1000 7200 950  7200
+Wire Wire Line
+	950  7200 950  7300
+Text Label 1600 6750 0    28   ~ 0
 12+
-NoConn ~ 5750 7300
-Text Label 5700 7400 0    28   ~ 0
+NoConn ~ 950  7300
+Text Label 900  7400 0    28   ~ 0
 12-
-Text Label 6050 7200 0    28   ~ 0
+Text Label 1250 7200 0    28   ~ 0
 12-
-NoConn ~ 6300 7200
-NoConn ~ 6050 7200
+NoConn ~ 1500 7200
+NoConn ~ 1250 7200
 Wire Wire Line
 	6200 1000 6200 1200
@@
 Connection ~ 3400 2750
 Wire Wire Line
-	3650 2650 3850 2650
-Wire Wire Line
-	3650 2850 3850 2850
+	3650 2650 3800 2650
+Wire Wire Line
+	3650 2850 3700 2850
 Text GLabel 4600 2650 2    50   Input ~ 0
 PC5
@@
 Wire Wire Line
 	9900 2200 10100 2200
+Text Notes 7050 6950 0    157  Italic 0
+AxoloRack - Another EurorAxoloti\n
+$Comp
+L power:VDD #PWR012
+U 1 1 5E1EE9E8
+P 4800 3100
+F 0 "#PWR012" H 4800 2950 50  0001 C CNN
+F 1 "VDD" H 4817 3273 50  0000 C CNN
+F 2 "" H 4800 3100 50  0001 C CNN
+F 3 "" H 4800 3100 50  0001 C CNN
+	1    4800 3100
+	1    0    0    -1
+$EndComp
+$Comp
+L Device:R R3
+U 1 1 5E1F014E
+P 4600 3200
+F 0 "R3" V 4550 3050 50  0000 C CNN
+F 1 "10K" V 4600 3200 50  0000 C CNN
+F 2 "" V 4530 3200 50  0001 C CNN
+F 3 "~" H 4600 3200 50  0001 C CNN
+	1    4600 3200
+	0    1    1    0
+$EndComp
+$Comp
+L Device:R R4
+U 1 1 5E1F6FE2
+P 4600 3350
+F 0 "R4" V 4550 3200 50  0000 C CNN
+F 1 "10K" V 4600 3350 50  0000 C CNN
+F 2 "" V 4530 3350 50  0001 C CNN
+F 3 "~" H 4600 3350 50  0001 C CNN
+	1    4600 3350
+	0    1    1    0
+$EndComp
+Wire Wire Line
+	4800 3100 4800 3200
+Wire Wire Line
+	4800 3200 4750 3200
+Wire Wire Line
+	4450 3200 3700 3200
+Wire Wire Line
+	3700 3200 3700 2850
+Connection ~ 3700 2850
+Wire Wire Line
+	3700 2850 3850 2850
+Wire Wire Line
+	4800 3200 4800 3350
+Wire Wire Line
+	4800 3350 4750 3350
+Connection ~ 4800 3200
+Wire Wire Line
+	4450 3350 3800 3350
+Wire Wire Line
+	3800 3350 3800 2650
+Connection ~ 3800 2650
+Wire Wire Line
+	3800 2650 3850 2650
 $EndSCHEMATC
